File: loconet.kicad_pcb (KiCad board)
At the start: 2 copper layers, 79.4 x 91.6 mm, 51 parts, among them CON1 BARREL_JACK, J1 RJ12, J2 RJ12, J3 RJ12, J4 RJ12, J5 RJ12, J6 RJ12, P1 CONN_01X04, P10 CONN_01X04, P2 CONN_01X04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

Commit message: Added github links to every module
Other:
- board text added: "http://bit.ly/1HuogNj"
