File: loconet.kicad_pcb (KiCad board)
At the start: 2 copper layers, 79.4 x 91.6 mm, 51 parts, among them CON1 BARREL_JACK, J1 RJ12, J2 RJ12, J3 RJ12, J4 RJ12, J5 RJ12, J6 RJ12, P1 CONN_01X04, P10 CONN_01X04, P2 CONN_01X04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

Commit message: Fixed LM317 footprint
Parts:
- U1: footprint Transistors_TO-220:TO-220_Neutral123_Vertical -> Regulators:LM317
Routing:
- net Loconet: track 297.4 -> 298.2 mm
Changed lines of the file:
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@@
-(kicad_pcb (version 4) (host pcbnew "(2015-05-08 BZR 5647)-product")
+(kicad_pcb (version 4) (host pcbnew "(2015-06-19 BZR 5795)-product")
   (general
     (links 104)
-    (no_connects 0)
+    (no_connects 3)
     (area 99.899999 58.515 200.100001 160.100001)
     (thickness 1.6)
     (drawings 51)
-    (tracks 279)
+    (tracks 283)
     (zones 0)
     (modules 51)
@@
       (at (xyz 0 0 0))
       (scale (xyz 0.4 0.4 0.4))
-      (rotate (xyz 0 0 0))
-    )
-  )
-  (module Transistors_TO-220:TO-220_Neutral123_Vertical (layer F.Cu)
-    (at 183.25 137)
-    (descr "TO-220, Neutral, Vertical,")
-    (tags "TO-220, Neutral, Vertical,")
-    (fp_text reference U1 (at 0 -5.08) (layer F.SilkS)
-      (effects (font (size 1 1) (thickness 0.15)))
-    )
-    (fp_text value LM317AT (at -3.75 2.75) (layer F.Fab)
-      (effects (font (size 1 1) (thickness 0.15)))
-    )
-    (fp_line (start -1.524 -3.048) (end -1.524 -1.905) (layer F.SilkS) (width 0.15))
-    (fp_line (start 1.524 -3.048) (end 1.524 -1.905) (layer F.SilkS) (width 0.15))
-    (fp_line (start 5.334 -1.905) (end 5.334 1.778) (layer F.SilkS) (width 0.15))
-    (fp_line (start 5.334 1.778) (end -5.334 1.778) (layer F.SilkS) (width 0.15))
-    (fp_line (start -5.334 1.778) (end -5.334 -1.905) (layer F.SilkS) (width 0.15))
-    (fp_line (start 5.334 -3.048) (end 5.334 -1.905) (layer F.SilkS) (width 0.15))
-    (fp_line (start 5.334 -1.905) (end -5.334 -1.905) (layer F.SilkS) (width 0.15))
-    (fp_line (start -5.334 -1.905) (end -5.334 -3.048) (layer F.SilkS) (width 0.15))
-    (fp_line (start 0 -3.048) (end -5.334 -3.048) (layer F.SilkS) (width 0.15))
-    (fp_line (start 0 -3.048) (end 5.334 -3.048) (layer F.SilkS) (width 0.15))
-    (pad 2 thru_hole oval (at 0 0 90) (size 2.49936 1.50114) (drill 1.00076) (layers *.Cu *.Mask F.SilkS)
-      (net 1 Loconet))
-    (pad 1 thru_hole oval (at -2.54 0 90) (size 2.49936 1.50114) (drill 1.00076) (layers *.Cu *.Mask F.SilkS)
-      (net 14 "Net-(R1-Pad2)"))
-    (pad 3 thru_hole oval (at 2.54 0 90) (size 2.49936 1.50114) (drill 1.00076) (layers *.Cu *.Mask F.SilkS)
-      (net 13 +12V))
-    (model Transistors_TO-220.3dshapes/TO-220_Neutral123_Vertical.wrl
-      (at (xyz 0 0 0))
-      (scale (xyz 0.3937 0.3937 0.3937))
       (rotate (xyz 0 0 0))
     )
@@
     (fp_line (start 0.35052 0.89916) (end 0.7493 1.89992) (layer F.SilkS) (width 0.15))
   )
+  (module Regulators:LM317 (layer F.Cu)
+    (at 183.25 137)
+    (tags TO-220)
+    (fp_text reference U1 (at 0 -5.08) (layer F.SilkS)
+      (effects (font (size 1 1) (thickness 0.15)))
+    )
+    (fp_text value LM317AT (at 0 3.81) (layer F.Fab)
+      (effects (font (size 1 1) (thickness 0.15)))
+    )
+    (fp_line (start -1.524 -3.048) (end -1.524 -1.905) (layer F.SilkS) (width 0.15))
+    (fp_line (start 1.524 -3.048) (end 1.524 -1.905) (layer F.SilkS) (width 0.15))
+    (fp_line (start 5.334 -1.905) (end 5.334 1.778) (layer F.SilkS) (width 0.15))
+    (fp_line (start 5.334 1.778) (end -5.334 1.778) (layer F.SilkS) (width 0.15))
+    (fp_line (start -5.334 1.778) (end -5.334 -1.905) (layer F.SilkS) (width 0.15))
+    (fp_line (start 5.334 -3.048) (end 5.334 -1.905) (layer F.SilkS) (width 0.15))
+    (fp_line (start 5.334 -1.905) (end -5.334 -1.905) (layer F.SilkS) (width 0.15))
+    (fp_line (start -5.334 -1.905) (end -5.334 -3.048) (layer F.SilkS) (width 0.15))
+    (fp_line (start 0 -3.048) (end -5.334 -3.048) (layer F.SilkS) (width 0.15))
+    (fp_line (start 0 -3.048) (end 5.334 -3.048) (layer F.SilkS) (width 0.15))
+    (pad 1 thru_hole oval (at 0 0 90) (size 2.49936 1.50114) (drill 1.00076) (layers *.Cu *.Mask F.SilkS)
+      (net 14 "Net-(R1-Pad2)"))
+    (pad 2 thru_hole oval (at -2.54 0 90) (size 2.49936 1.50114) (drill 1.00076) (layers *.Cu *.Mask F.SilkS)
+      (net 1 Loconet))
+    (pad 3 thru_hole oval (at 2.54 0 90) (size 2.49936 1.50114) (drill 1.00076) (layers *.Cu *.Mask F.SilkS)
+      (net 13 +12V))
+    (model Transistors_TO-220.3dshapes/TO-220_Neutral123_Vertical.wrl
+      (at (xyz 0 0 0))
+      (scale (xyz 0.3937 0.3937 0.3937))
+      (rotate (xyz 0 0 0))
+    )
+  )
   (gr_text http://bit.ly/1HuogNj (at 159 137) (layer B.SilkS)
     (effects (font (size 1 1) (thickness 0.15)) (justify mirror))
@@
   (segment (start 174.5 137.75) (end 175.25 137) (width 0.25) (layer F.Cu) (net 0))
   (segment (start 167.64 75.67) (end 167.695 75.67) (width 0.25) (layer F.Cu) (net 0) (status 30))
+  (segment (start 187.96 136.850209) (end 187.96 132.153998) (width 0.25) (layer F.Cu) (net 1))
+  (segment (start 187.96 132.153998) (end 182.548002 126.742) (width 0.25) (layer F.Cu) (net 1))
+  (segment (start 182.548002 126.742) (end 179.97763 126.742) (width 0.25) (layer F.Cu) (net 1))
+  (segment (start 179.97763 126.742) (end 178.9 126.742) (width 0.25) (layer F.Cu) (net 1))
+  (segment (start 183.75 140.42) (end 184.749489 139.420511) (width 0.25) (layer F.Cu) (net 1))
+  (segment (start 184.749489 139.420511) (end 185.389698 139.420511) (width 0.25) (layer F.Cu) (net 1))
+  (segment (start 185.389698 139.420511) (end 187.96 136.850209) (width 0.25) (layer F.Cu) (net 1))
+  (segment (start 180.71 137) (end 180.71 137.49911) (width 0.25) (layer F.Cu) (net 1))
+  (segment (start 180.71 137.49911) (end 183.63089 140.42) (width 0.25) (layer F.Cu) (net 1))
+  (segment (start 183.63089 140.42) (end 183.75 140.42) (width 0.25) (layer F.Cu) (net 1))
   (segment (start 176.36 102.762) (end 175.138 101.54) (width 0.25) (layer F.Cu) (net 1))
   (segment (start 175.138 101.54) (end 165.46 101.54) (width 0.25) (layer F.Cu) (net 1))
@@
   (segment (start 144.46 99) (end 144.46 112.5) (width 0.25) (layer B.Cu) (net 1))
   (segment (start 165.46 99) (end 165.46 112.5) (width 0.25) (layer F.Cu) (net 1))
-  (segment (start 183.25 139.92) (end 183.25 137) (width 0.25) (layer F.Cu) (net 1))
   (segment (start 183.75 140.42) (end 183.25 139.92) (width 0.25) (layer F.Cu) (net 1))
-  (segment (start 185.17 139) (end 186.25 139) (width 0.25) (layer F.Cu) (net 1))
-  (segment (start 186.25 139) (end 188 137.25) (width 0.25) (layer F.Cu) (net 1))
-  (segment (start 188 137.25) (end 188 131) (width 0.25) (layer F.Cu) (net 1))
-  (segment (start 188 131) (end 183.742 126.742) (width 0.25) (layer F.Cu) (net 1))
-  (segment (start 183.742 126.742) (end 178.9 126.742) (width 0.25) (layer F.Cu) (net 1))
-  (segment (start 183.75 140.42) (end 185.17 139) (width 0.25) (layer F.Cu) (net 1))
   (segment (start 142.71 128.75) (end 139 128.75) (width 0.25) (layer F.Cu) (net 1))
   (segment (start 139 128.75) (end 137 130.75) (width 0.25) (layer F.Cu) (net 1))
@@
   (segment (start 174.5 141.54986) (end 174.5 138.75) (width 0.25) (layer F.Cu) (net 13))
   (segment (start 172.25 136.5) (end 172.25 133) (width 0.25) (layer F.Cu) (net 13))
-  (segment (start 181.5 148.33) (end 181.5 137.79) (width 0.25) (layer F.Cu) (net 14))
-  (segment (start 181.5 137.79) (end 180.71 137) (width 0.25) (layer F.Cu) (net 14))
-  (segment (start 183.75 150.58) (end 181.5 148.33) (width 0.25) (layer F.Cu) (net 14))
+  (segment (start 183.75 150.58) (end 185.074491 149.255509) (width 0.25) (layer B.Cu) (net 14))
+  (segment (start 185.074491 149.255509) (end 185.074491 139.323601) (width 0.25) (layer B.Cu) (net 14))
+  (segment (start 185.074491 139.323601) (end 183.25 137.49911) (width 0.25) (layer B.Cu) (net 14))
+  (segment (start 183.25 137.49911) (end 183.25 137) (width 0.25) (layer B.Cu) (net 14))
   (zone (net 2) (net_name GND) (layer B.Cu) (hatch edge 0.508)
     (connect_pads (clearance 0.508))
